Commit message: Fix gripper collision box rotation and position, update Schunk xacro

File: joulin_vacuum_gripper/abb_gripper_description/urdf/pp_pg_160x600.urdf.xacro (robot description, xacro)
@@ -10,21 +10,7 @@
   Date:        2026-06-05
   ============================================================
-  Physical dimensions (from datasheet + STL bounding box):
-    Length: 600mm (X axis in mesh)
-    Width:  160mm (Z axis in mesh)
-    Height:  87mm (Y axis in mesh, origin at TOP = flange face)
-    Weight:  4.6 kg
-  STL coordinate system:
-    X: -300 to +300  (600mm length, centered)
-    Y:    0 to  +87  (87mm height, Y=0 is mounting face)
-    Z:  -80 to  +80  (160mm width, centered)
-    Top face normals point +Y
-  Visual rotation: rpy="${pi/2} ${pi} ${-pi/2}"
-    Maps STL to correct orientation with mounting face at tool parent
-  USAGE:
-    <xacro:include filename="$(find abb_gripper_description)/urdf/pp_pg_160x600.urdf.xacro"/>
-    <xacro:pp_pg_160x600 parent="rob1_swa_160_tool_mount" prefix="rob1_"/>
-  TO REMOVE: comment out those two lines.
-  TCP frame: rob1_gripper_tcp — 87mm forward from parent frame
+  STL: Y=0 mounting face, Y=+87 suction face
+  Visual xyz="0 0 0.087" — correct position, small gap is flange mesh depth
+  Collision: simple box, same position as visual, NO rotation needed
 -->
 <robot xmlns:xacro="http://www.ros.org/wiki/xacro">
@@ -42,14 +28,19 @@
       </visual>
       <collision>
-        <!-- Same rotation as visual so box aligns with mesh -->
-        <origin xyz="0 0 0.087" rpy="${pi/2} ${pi} ${-pi/2}"/>
+        <!--
+          Box in URDF frame (no rotation):
+            X = 0.600m (600mm length, horizontal)
+            Y = 0.160m (160mm width)
+            Z = 0.087m (87mm depth, forward from flange)
+          Center at half depth = 0.0435m forward from link origin
+        -->
+        <origin xyz="0 0 0.0435" rpy="0 0 ${pi/2}"/>
         <geometry>
-          <!-- In STL frame: X=600mm, Y=87mm depth, Z=160mm width -->
-          <box size="0.600 0.087 0.160"/>
+          <box size="0.600 0.160 0.087"/>
         </geometry>
       </collision>
       <inertial>
         <mass value="4.6"/>
-        <origin xyz="0 0 0.0435" rpy="0 0 0"/>
+        <origin xyz="0 0 0.0435" rpy="0 0 ${pi/2}"/>
         <inertia
           ixx="0.03481" ixy="0.0" ixz="0.0"

File: schunk_tool_changer/sws_160_description/urdf/sws_160.urdf.xacro (robot description, xacro)
@@ -10,25 +10,19 @@
   Date:        2026-06-05
   ============================================================
-  STL coordinate system (both parts):
-    Cylinder AXIS along Y
-    X: centered (-88 to +88)
-    Z: centered (-108.5 to +108.5)
-  SWK-160: Y=-30 (flange face) to Y=+70.6 (interface face)
-  SWA-160: Y=-37.5 (tool mount) to Y=0 (interface face)
-  Rotation needed: STL Y → tool0 Z = rpy="${-pi/2} 0 0"
-  Offsets (after rotation, STL Y becomes URDF Z):
-    SWK: flange face at STL Y=-30 → after rotation URDF Z=-30mm
-         → xyz="0 0 0.030" pushes mounting face to Z=0 (tool0)
-    SWA: interface face at STL Y=0 → after rotation URDF Z=0
-         → xyz="0 0 0" interface face already at Z=0
+  Rotation rpy="${pi/2} ${pi} ${-pi/2}" maps STL Y → URDF -Z
+  SWK-160: Y=-30 (flange face) to Y=+70.6 (interface) = 100.6mm
+    After rotation: flange face at URDF Z=+30, interface at URDF Z=-70.6
+    Visual offset = total_height - abs(Y_min) = 100.6 - 30 = 70.6mm
+    → xyz="0 0 0.0706" places flange face flush at link origin (Z=0)
+  SWA-160: Y=-37.5 (tool mount) to Y=0 (interface) = 37.6mm
+    After rotation: interface at URDF Z=0, tool mount at URDF Z=+37.5
+    Visual offset = abs(Y_min) = 37.5mm
+    → xyz="0 0 0.0375" places interface face flush at link origin (Z=0)
 -->
 <robot xmlns:xacro="http://www.ros.org/wiki/xacro">
-  <!-- ═══════════════════════════════════════════════════
-       SWK-160 ROBOT SIDE — always mounted on tool0
-       ═══════════════════════════════════════════════════ -->
   <xacro:macro name="swk_160_robot_side" params="parent prefix">
     <link name="${prefix}swk_160_link">
       <visual>
-        <origin xyz="0 0 0" rpy="${-pi/2} 0 0"/>
+        <origin xyz="0 0 0.0706" rpy="${pi/2} ${pi} ${-pi/2}"/>
         <geometry>
           <mesh filename="package://sws_160_description/meshes/swk_160_robot_side_bin.stl"
@@ -64,11 +58,8 @@
     </joint>
   </xacro:macro>
-  <!-- ═══════════════════════════════════════════════════
-       SWA-160 TOOL SIDE — permanently in URDF
-       ═══════════════════════════════════════════════════ -->
   <xacro:macro name="swa_160_tool_side" params="parent prefix">
     <link name="${prefix}swa_160_link">
       <visual>
-        <origin xyz="0 0 0" rpy="${-pi/2} 0 0"/>
+        <origin xyz="0 0 0.0375" rpy="${pi/2} ${pi} ${-pi/2}"/>
         <geometry>
           <mesh filename="package://sws_160_description/meshes/swa_160_tool_side_bin.stl"
